File: superDuino1.sch (EAGLE design)
At the start: 25 parts

Commit message: Added a BOM file and updated schematic and layout to address: Issue #7, Issue #6, Issue #5, Issue #4, Issue #3, Issue #2, Issue #1
Parts:
- removed JP4: M13, SparkFun-Connectors:M13
- removed X4: (no value), SparkFun-Connectors:DB25H
- added J1: POWER_JACKPTH, SparkFun-Connectors:POWER_JACKPTH
- added JP3: (no value), SparkFun-Connectors:ARDUINO_SERIAL_PROGRAMPTH
- added LED1, LED2, RX, TX: (no value), SparkFun-LED:LED1206
- added R1, R2, R3, R6, R7: (no value), rcl:R-US_R0805
- added R4, R5: SOLDERJUMPERNC, SparkFun-Retired:SOLDERJUMPERNC
- added S1: (no value), SparkFun-Electromechanical:TAC_SWITCHPTH
- C7: value 10uF -> (none); device rcl:C-US050-055X075 -> rcl:C-US050-035X075
- JP2: value M13 -> (none); device SparkFun-Connectors:M13 -> SparkFun-Connectors:M03X22X3_SILK_SM
Connections:
- net 1.5V renamed 1V5
- net DSTROBE renamed PMRW
- net N$10 renamed XA4
- net N$11 renamed XA16
- net N$12 renamed XA3
- net N$9 renamed XA17
- net RW renamed PMSTB
- net X2IO16 renamed XB16
- net X2IO17 renamed XB17
- net X2IO18 renamed XB18
- net X2IO19 renamed XB19
- net X2IO20 renamed XB20
- net X2IO22 renamed XB22
- net X2IO23 renamed XB23
- removed net 3.3V: C3.2, C5.2, C8.2, C9.+, U$1.AVDD, U$1.ENVREG, U$1.VDD, U$1.VDD_2, U$1.VDD_3, U$1.VDD_4, U$1.VDD_5, U$2.VCCIB0, U$2.VCCIB1, U$2.VCCIB2, U$2.VCCIB3, U$2.VMV0, U$2.VMV1, U$2.VMV2, U$2.VMV3, U$3.3.3V, U$5.OUT, U$6.IN, U$8.VCC, X3.23
- removed net 5V: C11.+, C2.1, U$3.5V, U$4.OUT, X3.11
- removed net AN0: U$1.PGEC2/AN6/RP6/CN24/RB6, U$3.A0, X1.21
- removed net AN1: U$1.PGED2/AN7/RP7/CN25/RB7, U$3.A1, X1.9
- removed net AN2: U$1.AN8/RP8/CN26/RB8, U$3.A2, X1.22
- removed net AN3: U$1.AN9/RP9/CN27/RB9, U$3.A3, X1.10
- removed net AN4: U$1.AN10/CVREF/CN28/PMA13/RB10, U$3.A4, X1.23
- removed net AN5: U$1.AN11/CN29/PMA12/RB11, U$3.A5, X1.11
- removed net AREF: U$1.PMA6/VREF+/CN42/RA10, U$3.AREF
- removed net BE: U$1.RP22/CN52/PMBE/RD3, U$2.GBB0/IO37RSB0
- removed net N$2 (its old number): U$2.GAA2/IO118UDB3, X1.8
- removed net N$6: U$2.GAC2/IO116UDB3, X1.6
- removed net N$7: U$2.IO116VDB3, X1.18
- removed net N$8: U$2.IO112PSB3, X1.5
- removed net PMA0: U$1.AN15/REFO/RP29/CN12/PMA0/RB15, U$2.GAA0/IO00RSB0
- removed net RAW: C1.1, C10.+, JP2.1, JP2.13, JP4.1, JP4.13, U$3.VIN, U$4.IN, U$5.IN, X1.1, X1.13, X1.14, X1.25, X2.1, X2.13, X2.14, X2.25, X3.1, X3.13, X3.14, X3.25, X4.1, X4.13, X4.14, X4.25
- removed net X2IO10: JP2.10, U$2.GEC2/IO95RSB2, X2.10
- removed net X2IO11: JP2.11, U$2.GEA2/IO97RSB2, X2.11
- removed net X2IO21: U$2.IO91RSB2, X2.21
- removed net X2IO3: JP2.3, U$2.GDA2/IO61RSB2, X2.3
- removed net X2IO4: JP2.4, U$2.GDC2/IO63RSB2, X2.4
- removed net X2IO5: JP2.5, U$2.IO74RSB2, X2.5
- removed net X2IO6: JP2.6, U$2.IO84RSB2, X2.6
- removed net X2IO7: JP2.7, U$2.IO86RSB2, X2.7
- removed net X2IO8: JP2.8, U$2.IO90RSB2, X2.8
- removed net X2IO9: JP2.9, U$2.IO92RSB2, X2.9
- removed net X4IO10: JP4.10, U$1.RP142/CN57/RD12, X4.10
- removed net X4IO11: JP4.11, U$1.C3INB/CN15/RD6, X4.11
- removed net X4IO16: U$1.OSCI/CLKI/CN23/RC12, X4.16
- removed net X4IO17: U$1.ASCL2/RP136/CN43/RA14, X4.17
- removed net X4IO18: U$1.RTCC/RP2/CN53/RD8, X4.18
- removed net X4IO19: U$1.RP3/CN55/PMCS2/RD10, X4.19
- removed net X4IO20: U$1.RP11/CN49/RD0, X4.20
- removed net X4IO21: U$1.SOSCO/C3INC/RP137/CN0/RC14, X4.21
- removed net X4IO22: U$1.RP23/CN51/RD2, X4.22
- removed net X4IO23: U$1.CN19/RD13, X4.23
- removed net X4IO3: JP4.3, U$1.TDO/CN38/RA5, X4.3
- removed net X4IO4: JP4.4, U$1.OSCO/CLKO/CN22/RC15, X4.4
- removed net X4IO5: JP4.5, U$1.ASDA2/RP135/CN44/RA15, X4.5
- removed net X4IO6: JP4.6, U$1.RP4/CN54/RD9, X4.6
- removed net X4IO7: JP4.7, U$1.RP12/CN56/PMCS1/RD11, X4.7
- removed net X4IO8: JP4.8, U$1.SOSCI/C3IND/CN1/RC13, X4.8
- removed net X4IO9: JP4.9, U$1.RP24/CN50/RD1, X4.9
- new net 3V3: C3.2, C5.2, C8.2, C9.+, JP2.2, JP3.VCC, R1.1, R3.1, R4.2, R5.2, R6.1, R7.1, U$1.AVDD, U$1.ENVREG, U$1.VDD, U$1.VDD_2, U$1.VDD_3, U$1.VDD_4, U$1.VDD_5, U$2.VCCIB0, U$2.VCCIB1, U$2.VCCIB2, U$2.VCCIB3, U$2.VMV0, U$2.VMV1, U$2.VMV2, U$2.VMV3, U$3.3.3V, U$5.OUT, U$6.IN, U$8.VCC
- new net 5V0: C11.+, C2.1, U$3.5V, U$4.OUT
- new net A0: U$1.AN8/RP8/CN26/RB8, U$3.A0
- new net A1: U$1.AN9/RP9/CN27/RB9, U$3.A1
- new net A2: U$1.AN10/CVREF/CN28/PMA13/RB10, U$3.A2
- new net A3: U$1.AN11/CN29/PMA12/RB11, U$3.A3
- new net A4: U$1.AN12/CTED2/CN30/PMA11/RB12, U$3.A4
- new net A5: U$1.AN13/CTED1/CN31/PMA10/RB13, U$3.A5
- new net N$1: LED1.A, R1.2
- new net PMA6: U$1.PMA6/VREF+/CN42/RA10, U$2.GAA0/IO00RSB0
- new net REFO: U$1.AN15/REFO/RP29/CN12/PMA0/RB15, U$2.GBB0/IO37RSB0
- new net VRAW: C1.1, C10.+, J1.PWR, U$3.VIN, U$4.IN, U$5.IN, X1.1, X1.13, X1.14, X1.25, X2.1, X2.13, X2.14, X2.25, X3.1, X3.13, X3.14, X3.25
- new net XA10: U$2.GAB2/IO117UDB3, X1.10
- new net XA11: U$2.GAA2/IO118UDB3, X1.11
- new net XA18: U$2.GFA2/IO107PSB3, X1.18
- new net XA19: U$2.GFA0/IO108NPB3, X1.19
- new net XA20: U$2.GFB1/IO109PDB3, X1.20
- new net XA21: U$2.IO116VDB3, X1.21
- new net XA22: U$2.IO117VDB3, X1.22
- new net XA23: U$2.IO118VDB3, X1.23
- new net XA5: U$2.GFC2/IO105PSB3, X1.5
- new net XA6: U$2.GFA1/IO108PPB3, X1.6
- new net XA7: U$2.GFB0/IO109NDB3, X1.7
- new net XA8: U$2.IO112PSB3, X1.8
- new net XA9: U$2.GAC2/IO116UDB3, X1.9
- new net XB10: U$2.GEC2/IO95RSB2, X2.10
- new net XB11: U$2.GEA2/IO97RSB2, X2.11
- new net XB21: LED2.A, U$2.IO91RSB2, X2.21
- new net XB3: U$2.GDA2/IO61RSB2, X2.3
- new net XB4: U$2.GDC2/IO63RSB2, X2.4
- new net XB5: U$2.IO74RSB2, X2.5
- new net XB6: U$2.IO84RSB2, X2.6
- new net XB7: U$2.IO86RSB2, X2.7
- new net XB8: U$2.IO90RSB2, X2.8
- new net XB9: U$2.IO92RSB2, X2.9
- new net XC10: U$2.GDC1/IO58UDB1, X3.10
- new net XC11: U$2.GDA1/IO60USB1, X3.11
- new net XC16: U$2.GBA0/IO39RSB0, X3.16
- new net XC17: U$2.GBA2/IO41PDB1, X3.17
- new net XC18: U$2.GBB2/IO42PSB1, X3.18
- new net XC19: U$2.IO43NDB1, X3.19
- new net XC20: U$2.GCA0/IO48NDB1, X3.20
- new net XC21: U$2.GCA1/IO50PDB1, X3.21
- new net XC22: U$2.IO52NDB1, X3.22
- new net XC23: U$2.GDC0/IO58VDB1, X3.23
- new net XC3: U$2.GBB1/IO38RSB0, X3.3
- new net XC4: U$2.GBA1/IO40RSB0, X3.4
- new net XC5: U$2.IO41NDB1, X3.5
- new net XC6: U$2.GBC2/IO42PDB1, X3.6
- new net XC7: U$2.GCC1/IO48PDB1, X3.7
- new net XC8: U$2.GCA0/IO50NDB1, X3.8
- new net XC9: U$2.GCB2/IO52PDB1, X3.9
- net D10: now also U$1.RP22/CN52/PMBE/RD3; no longer U$1.RP145/INT0/CN72/RF6, X3.8
- net D11: now also JP2.4, U$1.RP11/CN49/RD0; no longer U$1.SCL2/CN35/RA2, X3.21
- net D12: now also JP2.1, U$1.RP24/CN50/RD1; no longer U$1.SDA2/CN36/RA3, X3.9
- net D13: now also JP2.3, LED1.C, U$1.RP23/CN51/RD2; no longer U$1.TDI/CN37/RA4, X3.22
- net D2: now also U$1.RP17/CN18/PMA8/RF5; no longer U$1.RP143/CN20/RD14, X3.4
- net D3: now also U$1.RP16/CN7/RF3; no longer U$1.RP5/CN21/RD15, X3.17
- net D4: now also U$1.RP30/CN70/RF2; no longer U$1.RP10/CN17/PMA9/RF4, X3.5
- net D5: now also U$1.RP15/CN74/RF8; no longer U$1.RP17/CN18/PMA8/RF5, X3.18
- net D6: now also U$1.RTCC/RP2/CN53/RD8; no longer U$1.RP16/CN7/RF3, X3.6
- net D7: now also U$1.RP4/CN54/RD9; no longer U$1.RP30/CN70/RF2, X3.19
- net D8: now also U$1.RP3/CN55/PMCS2/RD10; no longer U$1.RP15/CN74/RF8, X3.7
- net D9: now also U$1.RP12/CN56/PMCS1/RD11; no longer U$1.RP144/CN73/RF7, X3.20
- net GND: now also J1.GND, J1.GNDBREAK, JP2.6, JP3.GND, R2.1, S1.1; no longer JP2.12, JP2.2, JP4.12, JP4.2, U$1.VREF-/CN41/PMA7/RA9, X3.10, X4.12, X4.15, X4.2, X4.24
- net N$3: now also LED2.C, R2.2; no longer U$2.IO118VDB3, X1.20
- net N$4: now also R7.2, TX.A; no longer U$2.GAB2/IO117UDB3, X1.7
- net N$5: now also R6.2, RX.A; no longer U$2.IO117VDB3, X1.19
- net RST: now also JP2.5, R3.2, S1.3, U$3.RES
- net RX: now also JP3.TXO, RX.C, U$1.RP5/CN21/RD15; no longer U$1.PGEC3/AN5/C1INA/RP18/CN7/RB5, X3.3
- net SCL: now also U$1.CN79/RG12; no longer U$1.SCL1/CN83/RG2
- net SDA: now also U$1.CN81/RG14; no longer U$1.SDA1/CN84/RG3
- net TX: now also JP3.RXI, TX.C, U$1.RP10/CN17/PMA9/RF4; no longer U$1.PGED3/AN4/C1INB/RP28/CN6/RB4, X3.16
- net VJTAG: now also R5.1
- net VPUMP: now also R4.1
Other:
- moved on the sheet: C7, JP1, U$1, U$3, U$8, X1, X2, X3
